File: Prototype1/hardware/prototype1/prototype1.sch (EAGLE design)
At the start: 58 parts, among them IC1 ICE40UL1K-CM36AITR1K, IC2 LDL112D33R, IC3 FT2232HL-REEL, IC4 93LC46BT-I_OT, IC5 M95010-WMN6P, U2 ESP-WROOM-32

Commit message: only FPGA left (I think) and a bunch of new reference material
Parts:
- removed PAIR_PORT: (no value), connector:M02LOCK
- added D1: (no value), passives:DIODESMA
- added DNPAIR1: (no value), darknet8:DARKNET_8_PAIR_CONNECTORPTH
- added J2: (no value), connector:M04X2
- added R13, R14: 100 K, passives:RESISTOR0805-RES
- added R15: 4.7K, passives:RESISTOR0805-RES
- added R16: 10K, passives:RESISTOR0805-RES
- added SHITTY_ADDON: SAO1, defcon:DC26_SHITTY_ADDON_CONNECTORPTH
- added U$7: SWITCH_TACTILETACTILE-2PIN, switches:SWITCH_TACTILETACTILE-2PIN
Connections:
- removed net DISPLAY_MISO: J1.9, U2.IO12
- removed net DISPLAY_MOSI: J1.6, U2.IO13
- removed net DISPLAY_SCK: J1.7, U2.IO14
- removed net PAIR_RX: PAIR_PORT.1, U2.IO16
- removed net PAIR_TX: PAIR_PORT.2, U2.IO17
- removed net SD_MISO: SDCARD.3, U2.IO19
- removed net SD_MOSI: SDCARD.2, U2.IO23
- removed net SD_SCK: SDCARD.4, U2.IO18
- new net DISPLAY_SD_MISO: J1.9, SDCARD.3, U2.IO19
- new net DISPLAY_SD_MOSI: J1.6, SDCARD.2, U2.IO23
- new net DISPLAY_SD_SCK: J1.7, SDCARD.4, U2.IO18
- new net JTAG_CLK: IC3.ADBUS0, U2.IO13
- new net JTAG_TDI: IC3.ADBUS1, U2.IO12
- new net JTAG_TDO: IC3.ADBUS2, U2.IO15
- new net JTAG_TMS: IC3.ADBUS3, U2.IO14
- new net N$14: D1.C, SHITTY_ADDON.VCC
- new net N$9: R15.1, U$7.A
- new net RXD-SPI_PROM_MOSI: IC3.BDBUS1, J2.1, J2.5
- new net SPI_PROM_CLK: IC5.C, J2.8, R14.1
- new net SPI_PROM_CS: IC3.BDBUS3, IC5.!S, R13.1
- new net SPI_PROM_MISO: IC3.BDBUS2, IC5.Q
- new net SPI_PROM_MOSI: IC5.D, J2.6
- new net TXD-SPI_PROM_CLK: IC3.BDBUS0, J2.3, J2.7
- net DISPLAY_BACKLIT: now also U2.IO16
- net DISPLAY_CS: now also U2.IO17; no longer U2.IO15
- net DISPLAY_DATA_CMD: now also U2.IO4
- net DISPLAY_RESET: now also U2.IO2
- net GND: now also DNPAIR1.GND, IC5.VSS, R14.2, R16.1, SHITTY_ADDON.GND
- net N$3: now also IC5.!W, R16.2, U$7.C; no longer U$1.VCC
- net PROG_RX: now also J2.4
- net PROG_TX: now also J2.2
- net SCL: now also DNPAIR1.SCL, SHITTY_ADDON.SCL
- net SDA: now also DNPAIR1.SDA, SHITTY_ADDON.SDA
- net TOUCH_CLK: now also U2.IO26
- net TOUCH_CS: now also U2.IO27
- net TOUCH_DATA_IN: now also U2.IO25
- net TOUCH_DATA_OUT: now also U2.IO33
- net TOUCH_IRQ: now also U2.IO32
- net VCC: now also D1.A, IC5.!HOLD, IC5.VCC, R13.2, R15.2, U$1.VCC
Other:
- note added: "HOLD is LOW, so connecting to VCC for now but need more investigation"
- note added: "puts W bar low writes are disabled, so when programming the SPI PROM we'll need to hold the button (for now)"

Commit message: starting dev board layout
Parts:
- removed C13: 0.1 uF, passives:C-USC0805
- added C22, C23, C24, C25, C28: 0.1 uf, passives:C-USC0805
- added C26, C27: 10 uf, passives:C-USC0805
- added EMIFILTER1: MEM2012S101RT, passives:MEM2012S101RT
- added J3, J4: (no value), connector:M10SILK_FEMALE_PTH
- added J5: (no value), connector:M04X2
- added LED4: fpga-prog-done, leds:LED3MM
- added R17: 10 K, passives:RESISTOR0805-RES
- added R18, R20: 100, passives:RESISTOR0805-RES
- added R19, R21: 56, passives:RESISTOR0805-RES
- added U$6: SWITCH_TACTILETACTILE-2PIN, switches:SWITCH_TACTILETACTILE-2PIN
- LED1: value (none) -> charging
- LED2: value (none) -> rx-led
- LED3: value (none) -> tx-led
- renumbered FL2 to EMIFILTER2
Connections:
- new net BARCODE: IC1.BARCODE, J3.7
- new net CRESET_B: IC1.CRESET_B, R17.1, U$6.C
- new net IO34: J5.6, U2.IO34
- new net IO35: J5.8, U2.IO35
- new net IOB0A: IC1.IOB_0A, J4.3
- new net IOB10A: IC1.IOB_10A, J4.6
- new net IOB3BG6: IC1.IOB_3B_G6, J4.2
- new net IOB4A: IC1.IOB_4A, J4.8
- new net IOB5B: IC1.IOB_5B, J3.1
- new net IOB6A: IC1.IOB_6A, J4.4
- new net IOB7BG5: IC1.IOB_7B_G5, J4.1
- new net IOB8AG4: IC1.IOB_8A_G4, J4.7
- new net IOB_1B: IC1.IOB_1B, J4.5
- new net IOT12AG1: IC1.IOT_21A_G1, J3.2
- new net IOT18B: IC1.IOT_18B, J3.3
- new net IOT19A: IC1.IOT_19A, J3.8
- new net IOT22BG0: IC1.IOT_22B_G0, J4.9
- new net IOT24B: IC1.IOT_24B, J3.4
- new net IOT27A: IC1.IOT_27A, J4.10
- new net IRLED: IC1.IRLED, J3.6
- new net N$10: LED4.A, R21.2
- new net N$15: FL1.OUT/IN, R18.2, R19.1
- new net N$16: FL1.IN/OUT, R20.1
- new net N$17: IC1.IOB_11B_CDONE, R21.1
- new net RBG1: IC1.RGB1, J3.5
- new net RBO0: IC1.RGB0, J3.9
- new net RGB2: IC1.RGB2, J3.10
- new net SENSORVN: J5.4, U2.SENSOR_VN
- new net SENSORVP: J5.2, U2.SENSOR_VP
- new net VCC-FPGA-PLL: C27.1, C28.1, IC1.VCC, IC1.VCCPLL, R20.2
- net ESP-EN: now also ESP-RST.C; no longer ESP-RST.A
- net GND: now also C2.2, C22.2, C23.2, C24.2, C25.2, C26.1, C27.2, C28.2, C3.2, CN1.2, EMIFILTER1.GND_1, EMIFILTER1.GND_2, ESP-RST.A, IC1.GND_1, IC1.GND_2, IC1.GND_LED, LED4.C, R19.2, U$6.A; no longer C13.2, ESP-RST.C
- net N$19: now also EMIFILTER1.OUT/IN; no longer FL1.OUT/IN
- net SPI_PROM_CLK: now also IC1.IOB_16A_SCK
- net SPI_PROM_CS: now also IC1.IOB_17B_SS
- net SPI_PROM_MISO: now also IC1.IOB_14A_SO
- net SPI_PROM_MOSI: now also IC1.IOB_15B_SI
- net VCC: now also C22.1, C23.1, C24.1, C25.1, C26.2, EMIFILTER1.IN/OUT, IC1.SPI_VCCIO1, IC1.VCCIO0, IC1.VCCIO2, R17.2, R18.1; no longer C13.1, FL1.IN/OUT
Other:
- note added: "FPGA says PLL must have its own ground. Don't know how to do that, so for now I'm connecting to board ground. Does it need its own power and gnd or just ground?"
- note added: "VCC"
- note added: "VCCIO0"
- note added: "VCCIO1"
- note added: "VCCIO2"
- note added: "probaly want to invert this so the LED only turns one while its configuring"
- note added: "voltage divider to lower the 3.3 V to between 1.14 and 1.26"
- moved on the sheet: ESP-RST, IC1
