File: Prototype1/hardware/prototype1/prototype1.sch (EAGLE design)
At the start: 60 parts, among them IC2 LDL112D33R, IC3 FT2232HL-REEL, IC4 93LC46BT-I_OT, IC5 M95010-WMN6P, J7 TMP BATTERY, U2 ESP-WROOM-32

Commit message: updated breakout board
Parts:
- added U$3: CMD_C0DE_LOGOCMD_CODE_LOGO_TOP_COPPER, logos:CMD_C0DE_LOGOCMD_CODE_LOGO_TOP_COPPER
Changed lines of the file:
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@@
 <?xml version="1.0" encoding="utf-8"?>
 <!DOCTYPE eagle SYSTEM "eagle.dtd">
-<eagle version="9.2.2">
+<eagle version="9.3.0">
 <drawing>
 <settings>
@@
 <part name="J8" library="connector" deviceset="M06" device="NO_SILK_YES_STOP"/>
 <part name="J1" library="connector" deviceset="M14" device=""/>
+<part name="U$3" library="logos" deviceset="CMD_C0DE_LOGO" device="CMD_CODE_LOGO_TOP_COPPER"/>
 </parts>
 <sheets>
@@
 </nets>
 </sheet>
+<sheet>
+<plain>
+</plain>
+<instances>
+<instance part="U$3" gate="G$1" x="35.56" y="50.8" smashed="yes"/>
+</instances>
+<busses>
+</busses>
+<nets>
+</nets>
+</sheet>

Commit message: adding docs
Parts:
- added C2, C3: 0.1 uF, passives:C-USC0805
- C6, C7: value 20 pF -> 27 pF
Connections:
- net GND: now also C2.1, C3.2
- net VCC: now also C2.2, C3.1
Changed lines of the file:
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@@
 <part name="IC3" library="ICs" deviceset="FT2232HL-REEL" device=""/>
 <part name="F1" library="crystals-timing" deviceset="ABLS-12.000MHZ-B4-T" device=""/>
-<part name="C6" library="passives" deviceset="C-US" device="C0805" value="20 pF"/>
-<part name="C7" library="passives" deviceset="C-US" device="C0805" value="20 pF"/>
+<part name="C6" library="passives" deviceset="C-US" device="C0805" value="27 pF"/>
+<part name="C7" library="passives" deviceset="C-US" device="C0805" value="27 pF"/>
 <part name="C8" library="passives" deviceset="C-US" device="C0805" value="0.1 uF"/>
 <part name="C9" library="passives" deviceset="C-US" device="C0805" value="3.3 uF"/>
@@
 <part name="J1" library="connector" deviceset="M14" device=""/>
 <part name="U$3" library="logos" deviceset="CMD_C0DE_LOGO" device="CMD_CODE_LOGO_TOP_COPPER"/>
+<part name="C2" library="passives" deviceset="C-US" device="C0805" value="0.1 uF"/>
+<part name="C3" library="passives" deviceset="C-US" device="C0805" value="0.1 uF"/>
 </parts>
 <sheets>
@@
 <attribute name="VALUE" x="133.35" y="94.742" size="1.778" layer="96" rot="R180"/>
 </instance>
+<instance part="C3" gate="G$1" x="22.86" y="149.86" smashed="yes" rot="R270">
+<attribute name="NAME" x="23.495" y="156.464" size="1.778" layer="95" rot="R270"/>
+<attribute name="VALUE" x="16.129" y="159.004" size="1.778" layer="96" rot="R270"/>
+</instance>
 </instances>
 <busses>
@@
 <label x="137.16" y="111.76" size="1.778" layer="95"/>
 </segment>
+<segment>
+<pinref part="C3" gate="G$1" pin="2"/>
+<wire x1="17.78" y1="149.86" x2="15.24" y2="149.86" width="0.1524" layer="91"/>
+<label x="15.24" y="149.86" size="1.778" layer="95"/>
+</segment>
 </net>
 <net name="VCC" class="0">
@@
 </segment>
 <segment>
-<pinref part="IC4" gate="G$1" pin="VCC"/>
-<wire x1="25.4" y1="137.16" x2="25.4" y2="147.32" width="0.1524" layer="91"/>
-<label x="25.4" y="144.78" size="1.778" layer="95" rot="R90"/>
-</segment>
-<segment>
 <pinref part="R7" gate="G$1" pin="2"/>
 <wire x1="33.02" y1="149.86" x2="33.02" y2="152.4" width="0.1524" layer="91"/>
@@
 <wire x1="134.62" y1="91.44" x2="139.7" y2="91.44" width="0.1524" layer="91"/>
 <label x="139.7" y="91.44" size="1.778" layer="95"/>
+</segment>
+<segment>
+<pinref part="IC4" gate="G$1" pin="VCC"/>
+<pinref part="C3" gate="G$1" pin="1"/>
+<wire x1="25.4" y1="137.16" x2="25.4" y2="149.86" width="0.1524" layer="91"/>
+<wire x1="25.4" y1="149.86" x2="25.4" y2="160.02" width="0.1524" layer="91"/>
+<junction x="25.4" y="149.86"/>
+<label x="25.4" y="160.02" size="1.778" layer="95"/>
 </segment>
 </net>
@@
 <sheet>
 <plain>
-<text x="71.12" y="93.98" size="1.778" layer="91">HOLD is LOW, so connecting
+<text x="81.28" y="109.22" size="1.778" layer="91">HOLD is LOW, so connecting
 to VCC for now but need
 more investigation</text>
@@
 <instances>
 <instance part="IC5" gate="G$1" x="38.1" y="83.82" smashed="yes">
-<attribute name="NAME" x="62.23" y="91.44" size="1.778" layer="95" align="center-left"/>
-<attribute name="VALUE" x="62.23" y="88.9" size="1.778" layer="96" align="center-left"/>
+<attribute name="NAME" x="44.45" y="93.98" size="1.778" layer="95" align="center-left"/>
+<attribute name="VALUE" x="44.45" y="88.9" size="1.778" layer="96" align="center-left"/>
 </instance>
 <instance part="R13" gate="G$1" x="22.86" y="88.9" smashed="yes" rot="R90">
@@
 <attribute name="NAME" x="-14.1986" y="67.31" size="1.778" layer="95" rot="R90"/>
 <attribute name="VALUE" x="-9.398" y="67.31" size="1.778" layer="96" rot="R90"/>
+</instance>
+<instance part="C2" gate="G$1" x="71.12" y="93.98" smashed="yes">
+<attribute name="NAME" x="72.136" y="94.615" size="1.778" layer="95"/>
+<attribute name="VALUE" x="72.136" y="89.789" size="1.778" layer="96"/>
 </instance>
 </instances>
@@
 <label x="-12.7" y="63.5" size="1.778" layer="95"/>
 </segment>
+<segment>
+<pinref part="C2" gate="G$1" pin="1"/>
+<wire x1="71.12" y1="96.52" x2="71.12" y2="99.06" width="0.1524" layer="91"/>
+<label x="71.12" y="99.06" size="1.778" layer="95"/>
+</segment>
 </net>
 <net name="SPI_PROM_MOSI" class="0">
@@
 <segment>
 <pinref part="IC5" gate="G$1" pin="VCC"/>
-<wire x1="66.04" y1="83.82" x2="71.12" y2="83.82" width="0.1524" layer="91"/>
-<label x="71.12" y="83.82" size="1.778" layer="95"/>
-</segment>
-<segment>
+<wire x1="66.04" y1="83.82" x2="66.04" y2="88.9" width="0.1524" layer="91"/>
+<pinref part="C2" gate="G$1" pin="2"/>
+<wire x1="66.04" y1="88.9" x2="71.12" y2="88.9" width="0.1524" layer="91"/>
+<wire x1="71.12" y1="88.9" x2="73.66" y2="88.9" width="0.1524" layer="91"/>
+<junction x="71.12" y="88.9"/>
+<label x="73.66" y="88.9" size="1.778" layer="95"/>
+</segment>
+<segment>
