File: Prototype1/hardware/prototype1/prototype1-with-charging-circut.sch (EAGLE design)
At the start: 60 parts, among them IC2 LDL112D33R, IC3 FT2232HL-REEL, IC4 93LC46BT-I_OT, IC5 M95010-WMN6P, J7 TMP BATTERY, U2 ESP-WROOM-32

Commit message: initial prototype board design complete will use this one on bantam
Parts:
- removed J6: (no value), connector:M02PTH
- removed J7: TMP BATTERY, connector:M02PTH
- removed J8: (no value), connector:M06NO_SILK_YES_STOP
- added C13, C22, C23, C24, C25, C28: 0.1 uf, passives:C-USC0805
- added C2, C3: 4.7 uF, passives:C-USC0805
- added C26, C27: 10 uf, passives:C-USC0805
- added CN1: (no value), connector:JST_2PIN-THM-RA
- added FL1: MEM2012S101RT, passives:MEM2012S101RT
- added IC1: ICE40UL1K-CM36AITR1K, FPGA:ICE40UL1K-CM36AITR1K
- added J3, J4: (no value), connector:M10SILK_FEMALE_PTH
- added LED1: charging, leds:LED0603
- added LED4: fpga-prog-done, leds:LED3MM
- added PROGRAMMER: SERIAL_4, connector:SERIAL_4
- added R17: 10 K, passives:RESISTOR0805-RES
- added R18, R20: 100, passives:RESISTOR0805-RES
- added R19, R21: 56, passives:RESISTOR0805-RES
- added R2, R3: (no value), passives:RESISTOR0805-RES
- added SDCARD: (no value), connector:M04PTH
- added U$3: XBP15SRV05W-G, passives:XBP15SRV05W-G
- added U$4: DS21984E, charging-ic:DS21984E
- added U$5: SWITCH_SPDT, switches:SWITCH_SPDT
- added U$6: SWITCH_TACTILETACTILE-2PIN, switches:SWITCH_TACTILETACTILE-2PIN
- R6: value 10 K -> 12 K
- U$7: value SWITCH_TACTILETACTILE-2PIN-NARROW -> SWITCH_TACTILETACTILE-2PIN; device switches:SWITCH_TACTILETACTILE-2PIN-NARROW -> switches:SWITCH_TACTILETACTILE-2PIN
Connections:
- new net BARCODE: IC1.BARCODE, J3.7
- new net CRESET_B: IC1.CRESET_B, R17.1, U$6.C
- new net IOB0A: IC1.IOB_0A, J4.3
- new net IOB10A: IC1.IOB_10A, J4.6
- new net IOB3BG6: IC1.IOB_3B_G6, J4.2
- new net IOB4A: IC1.IOB_4A, J4.8
- new net IOB5B: IC1.IOB_5B, J3.1
- new net IOB6A: IC1.IOB_6A, J4.4
- new net IOB7BG5: IC1.IOB_7B_G5, J4.1
- new net IOB8AG4: IC1.IOB_8A_G4, J4.7
- new net IOB_1B: IC1.IOB_1B, J4.5
- new net IOT12AG1: IC1.IOT_21A_G1, J3.2
- new net IOT18B: IC1.IOT_18B, J3.3
- new net IOT19A: IC1.IOT_19A, J3.8
- new net IOT22BG0: IC1.IOT_22B_G0, J4.9
- new net IOT24B: IC1.IOT_24B, J3.4
- new net IOT27A: IC1.IOT_27A, J4.10
- new net IRLED: IC1.IRLED, J3.6
- new net N$1: LED1.A, R2.1
- new net N$10: LED4.A, R21.2
- new net N$15: FL1.OUT/IN, R18.2, R19.1
- new net N$16: FL1.IN/OUT, R20.1
- new net N$17: IC1.IOB_11B_CDONE, R21.1
- new net N$2: LED1.C, U$4.STAT
- new net N$4: R3.2, U$4.PROG
- new net N$5: C4.1, IC2.VIN, RESETTABLE_FUSE.2, U$5.2
- new net RBG1: IC1.RGB1, J3.5
- new net RBO0: IC1.RGB0, J3.9
- new net RGB2: IC1.RGB2, J3.10
- new net VCC-FPGA-PLL: C27.1, C28.1, IC1.VCC, IC1.VCCPLL, R20.2
- new net VCC5: C2.1, R2.2, U$2.+5V, U$4.VDD
- net DISPLAY_BACKLIT: now also J1.8; no longer J1.4
- net DISPLAY_CS: now also J1.3; no longer J1.5
- net DISPLAY_DATA_CMD: now also J1.5; no longer J1.3
- net DISPLAY_RESET: now also J1.4; no longer J1.2
- net DISPLAY_SD_MISO: now also J1.9, SDCARD.3; no longer J1.8
- net DISPLAY_SD_MOSI: now also J1.6, SDCARD.2; no longer J1.13
- net DISPLAY_SD_SCK: now also SDCARD.4
- net GND: now also C13.2, C2.2, C22.2, C23.2, C24.2, C25.2, C26.1, C27.2, C28.2, C3.2, CN1.2, FL1.GND_1, FL1.GND_2, IC1.GND_1, IC1.GND_2, IC1.GND_LED, J1.2, LED4.C, PROGRAMMER.GND, R19.2, R3.1, U$3.P2, U$4.VSS, U$5.1, U$6.A; no longer J1.14, J6.1, J7.1, J8.3
- net N$12: now also U$5.C; no longer C4.1, IC2.VIN, J6.2, RESETTABLE_FUSE.2
- net PROG_RX: now also J2.4, PROGRAMMER.TX; no longer J1.10
- net PROG_TX: now also J2.2, PROGRAMMER.RX; no longer J1.11
- net SCL: no longer J1.12
- net SDA: no longer J1.9
- net SD_CS: now also SDCARD.1; no longer J1.6
- net SPI_PROM_CLK: now also IC1.IOB_16A_SCK
- net SPI_PROM_CS: now also IC1.IOB_17B_SS
- net SPI_PROM_MISO: now also IC1.IOB_14A_SO
- net SPI_PROM_MOSI: now also IC1.IOB_15B_SI
- net TOUCH_CLK: now also J1.10; no longer J8.2
- net TOUCH_CS: now also J1.11; no longer J8.1
- net TOUCH_DATA_IN: now also J1.12; no longer J8.4
- net TOUCH_DATA_OUT: now also J1.13; no longer J8.5
- net TOUCH_IRQ: now also J1.14; no longer J8.6
- net USB_DM: now also U$3.P6
- net USB_DP: now also U$3.P1
- net VBAT: now also C3.1, CN1.1, U$4.VBAT; no longer J7.2
- net VCC: now also C13.1, C22.1, C23.1, C24.1, C25.1, C26.2, IC1.SPI_VCCIO1, IC1.VCCIO0, IC1.VCCIO2, IC1.VPP2V5, PROGRAMMER.VCC, R17.2, R18.1; no longer J5.7
Other:
- note added: "FPGA says PLL must have its own ground. Don't know how to do that, so for now I'm connecting to board ground. Does it need its own power and gnd or just ground?"
- note added: "For this prototype leaving off charging circut"
- note added: "VCC"
- note added: "VCCIO0"
- note added: "VCCIO1"
- note added: "VCCIO2"
- note added: "probaly want to invert this so the LED only turns one while its configuring"
- note added: "voltage divider to lower the 3.3 V to between 1.14 and 1.26"
- note removed: "For this prototype leaving off charging circut also leaving off usb diode so right now usb is just data not power! also leaving off power switch, will make it a jumper instead"
- moved on the sheet: J1
