File: Prototype1/hardware/prototype1/prototype1-ftdi-as-breakout.sch (EAGLE design)
At the start: 31 parts, among them IC2 LDL112D33R, IC5 M95010-WMN6P, J7 TMP BATTERY, U2 ESP-WROOM-32

Commit message: added logo and fixed drc error
Parts:
- added U$2: CMD_C0DE_LOGOCMD_CODE_LOGO_TOP_COPPER, logos:CMD_C0DE_LOGOCMD_CODE_LOGO_TOP_COPPER
Changed lines of the file:
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@@
 <part name="R3" library="passives" deviceset="RESISTOR" device="0805-RES" value="100"/>
 <part name="J8" library="connector" deviceset="M06" device="SILK_FEMALE_PTH"/>
+<part name="U$2" library="logos" deviceset="CMD_C0DE_LOGO" device="CMD_CODE_LOGO_TOP_COPPER"/>
 </parts>
 <sheets>
@@
 </nets>
 </sheet>
+<sheet>
+<plain>
+</plain>
+<instances>
+<instance part="U$2" gate="G$1" x="40.64" y="40.64" smashed="yes"/>
+</instances>
+<busses>
+</busses>
+<nets>
+</nets>
+</sheet>
