File: Prototype1/hardware/ft2232H Breakout/ft2232h-breakout.sch (EAGLE design)
At the start: 41 parts, among them IC2 LDL112D33R, IC3 FT2232HL-REEL, IC4 93LC46BT-I_OT

Commit message: updated breakout board
Parts:
- added J2, J3, J4, J5: (no value), connector:M15
- added LED1: (no value), leds:LED3MM
- added R1: 100 ohm, passives:RESISTORKIT
- added S1: (no value), switches:SWITCH-SPSTPTH
- J1: device connector:M04X2 -> connector:M02PTH
Connections:
- removed net N$18: C18.1, C19.1, EMIFILTER2.OUT/IN, IC3.VPLL
- removed net N$19: C20.1, C21.1, EMIFILTER1.OUT/IN, IC3.VPHY
- removed net N$7: IC3.REF, R6.1
- removed net RXD-SPI_PROM_MOSI: IC3.BDBUS1
- removed net SPI_PROM_CS: IC3.BDBUS3
- removed net SPI_PROM_MISO: IC3.BDBUS2
- removed net TXD-SPI_PROM_CLK: IC3.BDBUS0
- new net ACBUS0: IC3.ACBUS0, J3.6
- new net ACBUS1: IC3.ACBUS1, J3.5
- new net ACBUS2: IC3.ACBUS2, J3.4
- new net ACBUS3: IC3.ACBUS3, J3.3
- new net ACBUS4: IC3.ACBUS4, J3.2
- new net ACBUS5: IC3.ACBUS5, J3.1
- new net ACBUS6: IC3.ACBUS6, J4.3
- new net ACBUS7: IC3.ACBUS7, J4.4
- new net ADBUS4: IC3.ADBUS4, J3.11
- new net ADBUS5: IC3.ADBUS5, J3.10
- new net ADBUS6: IC3.ADBUS6, J3.9
- new net ADBUS7: IC3.ADBUS7, J3.8
- new net BCBUS0: IC3.BCBUS0, J4.15
- new net BCBUS1: IC3.BCBUS1, J5.8
- new net BCBUS2: IC3.BCBUS2, J5.9
- new net BCBUS5: IC3.BCBUS5, J5.13
- new net BCBUS6: IC3.BCBUS6, J5.14
- new net BDBUS0: IC3.BDBUS0, J4.5
- new net BDBUS1: IC3.BDBUS1, J4.6
- new net BDBUS2: IC3.BDBUS2, J4.7
- new net BDBUS3: IC3.BDBUS3, J4.8
- new net BDBUS4: IC3.BDBUS4, J4.10
- new net BDBUS5: IC3.BDBUS5, J4.11
- new net BDBUS6: IC3.BDBUS6, J4.12
- new net BDBUS7: IC3.BDBUS7, J4.13
- new net N$1: LED1.A, R1.1
- new net N$2: C4.1, IC2.VIN, R1.2, RESETTABLE_FUSE.2
- new net REF: IC3.REF, J2.11, R6.1
- new net VCC5: S1.S, U$2.+5V
- new net VIN: RESETTABLE_FUSE.1, S1.P
- new net VPHY: C20.1, C21.1, EMIFILTER1.OUT/IN, IC3.VPHY, J2.12
- new net VPLL: C18.1, C19.1, EMIFILTER2.OUT/IN, IC3.VPLL, J2.8
- net GND: now also J1.2, J2.15, J3.7, J4.14, J4.2, J5.4, J5.7
- net JTAG_CLK: now also J2.5
- net JTAG_TDI: now also J3.15
- net JTAG_TDO: now also J3.14
- net JTAG_TMS: now also J3.13
- net N$12: now also LED1.C; no longer C4.1, IC2.VIN, RESETTABLE_FUSE.2
- net OSCI: now also J2.14
- net OSCO: now also J2.13
- net RXD_LED: now also J5.10
- net TXD_LED: now also J5.11
- net USB_DM: now also J2.9
- net USB_DP: now also J2.10
- net VBAT: now also J1.1, S1.O; no longer RESETTABLE_FUSE.1
- net VCC: now also J2.3, J2.6, J3.12, J4.1, J4.9, J5.12, J5.15, J5.5
- net VCC1.8: now also J2.7, J5.6
