File: Prototype1/hardware/ft2232H Breakout/ft2232h-breakout-with-ground-planesch.brd (EAGLE design)
At the start: 78 x 91.5 mm, 48 parts, among them IC2 LDL112D33R, IC3 FT2232HL-REEL, IC4 93LC46BT-I_OT

Commit message: adding docs
Routing:
- net VCC1.8: track 131.5 -> 132.1 mm
Changed lines of the file:
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@@
 <wire x1="32.5687" y1="54.30835" x2="32.5687" y2="55.1133" width="0.1778" layer="1"/>
 <wire x1="32.5687" y1="55.1133" x2="32.46" y2="55.222" width="0.1778" layer="1"/>
-<polygon width="0.1524" layer="16" isolate="1.778">
+<polygon width="0.1524" layer="16" isolate="1.9304">
 <vertex x="0" y="99.9744"/>
 <vertex x="0" y="8.5344"/>
@@
 <wire x1="40.469" y1="70.231" x2="40.6282" y2="70.231" width="0.1778" layer="1"/>
 <wire x1="45.2628" y1="60.1472" x2="45.2628" y2="55.0164" width="0.1778" layer="16"/>
-<wire x1="29.3053" y1="74.010875" x2="29.662475" y2="73.6537" width="0.1778" layer="16"/>
-<wire x1="26.67" y1="78.74" x2="29.3053" y2="76.1047" width="0.1778" layer="16"/>
-<wire x1="31.7563" y1="73.6537" x2="36.4744" y2="68.9356" width="0.1778" layer="16"/>
+<wire x1="28.6957" y1="73.706075" x2="29.510075" y2="72.8917" width="0.1778" layer="16"/>
+<wire x1="26.67" y1="78.74" x2="28.6957" y2="76.7143" width="0.1778" layer="16"/>
+<wire x1="32.5183" y1="72.8917" x2="36.4744" y2="68.9356" width="0.1778" layer="16"/>
 <wire x1="36.4744" y1="68.9356" x2="45.2628" y2="60.1472" width="0.1778" layer="16"/>
-<wire x1="29.3053" y1="76.1047" x2="29.3053" y2="74.010875" width="0.1778" layer="16"/>
-<wire x1="29.662475" y1="73.6537" x2="31.7563" y2="73.6537" width="0.1778" layer="16"/>
+<wire x1="28.6957" y1="76.7143" x2="28.6957" y2="73.706075" width="0.1778" layer="16"/>
+<wire x1="29.510075" y1="72.8917" x2="32.5183" y2="72.8917" width="0.1778" layer="16"/>
 <wire x1="27.69953125" y1="56.2262" x2="27.7274" y2="56.2262" width="0.1778" layer="1"/>
 <wire x1="27.7274" y1="56.2262" x2="28.0416" y2="56.5404" width="0.1778" layer="1"/>
