File: Prototype1/hardware/prototype2/prototype2.brd (EAGLE design)
At the start: 101.6 x 75.9 mm, 94 parts, among them IC1 ATTINY13A-SSU, IC2 LDL112D33R, IC3 FT2232HL-REEL, IC4 93LC46BT-I_OT, IC5 APA104, IC6 APA104, IC7 APA104, IC8 APA104, J4 DN PAIR, U2 ESP-WROOM-32

Commit message: fixed bug with center ground plane on esp32
Connections:
- net GND: now also U2.GND
Changed lines of the file:
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@@
 <wire x1="19.84666875" y1="31" x2="21.4867" y2="29.35996875" width="0.1778" layer="1"/>
 <wire x1="18.582" y1="31" x2="19.84666875" y2="31" width="0.1778" layer="1"/>
+<contactref element="U2" pad="GND"/>
 </signal>
 <signal name="DISPLAY_CS">

Commit message: removed inputs to output pins....duh
Parts:
- removed R23, R24: 10 K, passives:0805
Connections:
- net PWRSAV: no longer R24.2
- net SUSPEND: no longer R23.2
- net VCC: no longer R23.1, R24.1
Routing:
- net PWRSAV: track 9.56 -> 0.00 mm
- net VCC: track 556.2 -> 547.3 mm
- net SUSPEND: track 3.97 -> 0.00 mm
- net GND: track 45.1 -> 43.6 mm
Changed lines of the file:
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@@
 <attribute name="VALUE" x="26.367" y="14.384" size="0.4064" layer="27" rot="R90"/>
-</element>
-<element name="R23" library="passives" package="0805" value="10 K" x="16.18" y="39.51" smashed="yes" rot="R270">
-<attribute name="NAME" x="17.0055" y="40.272" size="0.4064" layer="25" rot="R270"/>
-<attribute name="VALUE" x="14.783" y="40.526" size="0.4064" layer="27" rot="R270"/>
-</element>
-<element name="R24" library="passives" package="0805" value="10 K" x="24.42" y="18.53" smashed="yes" rot="R90">
-<attribute name="NAME" x="23.4945" y="18.418" size="0.4064" layer="25" rot="R90"/>
-<attribute name="VALUE" x="25.817" y="17.514" size="0.4064" layer="27" rot="R90"/>
 </element>
 <element name="R3" library="passives" package="0805" value="20 R" x="87.8" y="22.05" smashed="yes" rot="R180">
@@
 <contactref element="EMIFILTER1" pad="1"/>
 <contactref element="EMIFILTER2" pad="1"/>
-<contactref element="R23" pad="1"/>
-<contactref element="R24" pad="1"/>
 <contactref element="IC4" pad="6"/>
 <contactref element="C3" pad="1"/>
@@
 <wire x1="23.37" y1="25.73" x2="23.35" y2="25.75" width="0.254" layer="1"/>
 <wire x1="23.35" y1="25.75" x2="22.8" y2="25.2" width="0.254" layer="1"/>
-<wire x1="22.8" y1="25.2" x2="22.8" y2="17.55" width="0.254" layer="1"/>
-<wire x1="22.8" y1="17.55" x2="22.8" y2="1.65" width="0.254" layer="1"/>
+<wire x1="22.8" y1="25.2" x2="22.8" y2="1.65" width="0.254" layer="1"/>
 <wire x1="19.04" y1="23.94" x2="19.04" y2="21.24" width="0.254" layer="1"/>
 <wire x1="17.8" y1="20" x2="12.05" y2="20" width="0.254" layer="1"/>
@@
 <wire x1="24" y1="45" x2="24" y2="46" width="0.254" layer="1"/>
 <wire x1="24" y1="46" x2="23.05" y2="46.95" width="0.254" layer="1"/>
-<wire x1="23.05" y1="46.95" x2="18" y2="46.95" width="0.254" layer="1"/>
-<wire x1="18" y1="46.95" x2="16.18" y2="45.13" width="0.254" layer="1"/>
-<wire x1="16.18" y1="45.13" x2="16.18" y2="40.41" width="0.254" layer="1"/>
 <wire x1="4.74" y1="45.58" x2="6.11" y2="46.95" width="0.254" layer="1"/>
-<wire x1="6.11" y1="46.95" x2="18" y2="46.95" width="0.254" layer="1"/>
+<wire x1="6.11" y1="46.95" x2="23.05" y2="46.95" width="0.254" layer="1"/>
 <wire x1="41.3" y1="73.43" x2="41.24" y2="73.37" width="0.254" layer="1"/>
 <wire x1="41.24" y1="73.37" x2="36.25" y2="73.37" width="0.254" layer="1"/>
@@
 <wire x1="83.75" y1="59.47" x2="80.93" y2="62.29" width="0.254" layer="1"/>
 <wire x1="80.93" y1="62.29" x2="80.93" y2="62.44" width="0.254" layer="1"/>
-<wire x1="24.42" y1="17.63" x2="24.34" y2="17.55" width="0.1778" layer="1"/>
-<wire x1="24.34" y1="17.55" x2="22.8" y2="17.55" width="0.1778" layer="1"/>
 <wire x1="35.65" y1="13" x2="43" y2="13" width="0.254" layer="1"/>
 <wire x1="50" y1="20" x2="50" y2="25" width="0.254" layer="1"/>
@@
 <wire x1="24.1533" y1="39.14003125" x2="26.79333125" y2="36.5" width="0.1778" layer="1"/>
 <wire x1="26.79333125" y1="36.5" x2="30.058" y2="36.5" width="0.1778" layer="1"/>
-<wire x1="15.46953125" y1="39.2767" x2="16.89046875" y2="39.2767" width="0.1778" layer="1"/>
-<wire x1="17.5778" y1="37.23953125" x2="17.73403125" y2="37.0833" width="0.1778" layer="1"/>
-<wire x1="17.73403125" y1="37.0833" x2="18.4987" y2="37.0833" width="0.1778" layer="1"/>
-<wire x1="18.4987" y1="37.0833" x2="18.582" y2="37" width="0.1778" layer="1"/>
-<wire x1="14.26" y1="38.36" x2="14.55283125" y2="38.36" width="0.1778" layer="1"/>
-<wire x1="14.55283125" y1="38.36" x2="15.46953125" y2="39.2767" width="0.1778" layer="1"/>
-<wire x1="16.89046875" y1="39.2767" x2="17.5778" y2="38.58936875" width="0.1778" layer="1"/>
-<wire x1="17.5778" y1="38.58936875" x2="17.5778" y2="37.23953125" width="0.1778" layer="1"/>
 <wire x1="21.4867" y1="29.35996875" x2="21.4867" y2="28.5953" width="0.1778" layer="1"/>
 <wire x1="21.4867" y1="28.5953" x2="21.57" y2="28.512" width="0.1778" layer="1"/>
@@
 <wire x1="18.582" y1="31" x2="19.84666875" y2="31" width="0.1778" layer="1"/>
 <contactref element="U2" pad="GND"/>
+<wire x1="18.582" y1="37" x2="17" y2="37" width="0.1778" layer="1"/>
+<wire x1="15.64" y1="38.36" x2="14.26" y2="38.36" width="0.1778" layer="1"/>
+<wire x1="17" y1="37" x2="15.64" y2="38.36" width="0.1778" layer="1"/>
 </signal>
 <signal name="DISPLAY_CS">
@@
 <signal name="SUSPEND">
 <contactref element="IC3" pad="36"/>
-<contactref element="R23" pad="2"/>
-<wire x1="18.582" y1="36.5" x2="17.1" y2="36.5" width="0.254" layer="1"/>
-<wire x1="16.18" y1="37.42" x2="16.18" y2="38.61" width="0.254" layer="1"/>
-<wire x1="17.1" y1="36.5" x2="16.18" y2="37.42" width="0.254" layer="1"/>
 </signal>
 <signal name="PWRSAV">
 <contactref element="IC3" pad="59"/>
-<contactref element="R24" pad="2"/>
-<wire x1="25.57" y1="20.63865" x2="24.42" y2="19.48865" width="0.254" layer="1"/>
-<wire x1="24.42" y1="19.43" x2="24.42" y2="19.48865" width="0.254" layer="1"/>
-<wire x1="25.57" y1="20.63865" x2="25.57" y2="28.512" width="0.254" layer="1"/>
 </signal>
 <signal name="RXD_SPI_PROM_MOSI">
